File: hardware/tl494.brd (EAGLE design)
At the start: 100 x 80 mm, 72 parts, among them IC1 TL494CN, K1 24V, Q1 2N5551, Q1I 8050, Q2 8550, Q2I 8050, Q3 8050, Q4 2SK4145, Q5 2SK4145

Commit message: minor update
Parts:
- R12: device rcl:0207/10 -> rcl:0207/5V
- moved R7 85.4 mm to (40.6, 58.4)
- moved R6 65.4 mm to (33.0, 57.1), turned to 90 degrees
- moved C2 8.13 mm to (21.6, 50.8), turned to 0 degrees

Commit message: added turn on latch circuit and gitignore
Parts:
- added C17: 1uF 63V, rcl:E3,5-10
- added Q1I1: 2N3904, dp_devices.v6:TO-92
- added Q6: IRF9530, transistor-power:TO220BV
- added R34: 50K, rcl:0207/10
- added R35, R36, R37: 100K, rcl:0207/10
- added SW1: SW_MEMBRANE, dp_devices.v6:SW_MEMBRANE
Connections:
- new net N$29: Q6.S, R36.1, R37.1
- new net N$30: Q6.G, R34.2, R36.2
- new net N$31: Q1I1.3, R34.1
- new net N$32: Q6.D, R35.2
- new net N$33: C17.+, Q1I1.2, R35.1, SW1.P$1
- new net N$34: R37.2, SW1.P$2
- net GND: now also C17.-, Q1I1.1
Changed lines of the file:
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@@
 <?xml version="1.0" encoding="utf-8"?>
 <!DOCTYPE eagle SYSTEM "eagle.dtd">
-<eagle version="9.1.3">
+<eagle version="9.4.2">
 <drawing>
 <settings>
@@
 <attribute name="VALUE" x="-52.705" y="0.9525" size="1.27" layer="27" ratio="10"/>
 </element>
+<element name="Q6" library="transistor-power" library_urn="urn:adsk.eagle:library:400" package="TO220BV" package3d_urn="urn:adsk.eagle:package:29484/3" value="IRF9530" x="-82.55" y="0" smashed="yes">
+<attribute name="NAME" x="-87.63" y="-6.0452" size="1.27" layer="25" ratio="10"/>
+<attribute name="VALUE" x="-87.63" y="-7.62" size="1.27" layer="27" ratio="10"/>
+</element>
+<element name="R34" library="rcl" library_urn="urn:adsk.eagle:library:334" package="0207/10" package3d_urn="urn:adsk.eagle:package:23491/2" value="50K" x="-82.55" y="-12.7" smashed="yes">
+<attribute name="NAME" x="-85.598" y="-11.176" size="1.27" layer="25" ratio="10"/>
+<attribute name="SPICEPREFIX" value="R" x="-82.55" y="-12.7" size="1.778" layer="27" display="off"/>
+<attribute name="VALUE" x="-84.8106" y="-13.335" size="1.27" layer="27" ratio="10"/>
+</element>
+<element name="Q1I1" library="dp_devices.v6" package="TO-92" value="2N3904" x="-93.98" y="-8.89" smashed="yes">
+<attribute name="NAME" x="-96.52" y="-5.842" size="1.27" layer="25" font="vector" ratio="10"/>
+<attribute name="VALUE" x="-96.52" y="-12.192" size="1.27" layer="27" font="vector" ratio="10"/>
+</element>
+<element name="R35" library="rcl" library_urn="urn:adsk.eagle:library:334" package="0207/10" package3d_urn="urn:adsk.eagle:package:23491/2" value="100K" x="-91.44" y="-17.78" smashed="yes">
+<attribute name="NAME" x="-94.488" y="-16.256" size="1.27" layer="25" ratio="10"/>
+<attribute name="SPICEPREFIX" value="R" x="-91.44" y="-17.78" size="1.778" layer="27" display="off"/>
+<attribute name="VALUE" x="-93.7006" y="-18.415" size="1.27" layer="27" ratio="10"/>
+</element>
+<element name="R36" library="rcl" library_urn="urn:adsk.eagle:library:334" package="0207/10" package3d_urn="urn:adsk.eagle:package:23491/2" value="100K" x="-91.44" y="-22.86" smashed="yes">
+<attribute name="NAME" x="-94.488" y="-21.336" size="1.27" layer="25" ratio="10"/>
+<attribute name="SPICEPREFIX" value="R" x="-91.44" y="-22.86" size="1.778" layer="27" display="off"/>
+<attribute name="VALUE" x="-93.7006" y="-23.495" size="1.27" layer="27" ratio="10"/>
+</element>
+<element name="R37" library="rcl" library_urn="urn:adsk.eagle:library:334" package="0207/10" package3d_urn="urn:adsk.eagle:package:23491/2" value="100K" x="-91.44" y="-27.94" smashed="yes">
+<attribute name="NAME" x="-94.488" y="-26.416" size="1.27" layer="25" ratio="10"/>
+<attribute name="SPICEPREFIX" value="R" x="-91.44" y="-27.94" size="1.778" layer="27" display="off"/>
+<attribute name="VALUE" x="-93.7006" y="-28.575" size="1.27" layer="27" ratio="10"/>
+</element>
+<element name="SW1" library="dp_devices.v6" package="SW_MEMBRANE" value="SW_MEMBRANE" x="-101.6" y="-25.4" smashed="yes">
+<attribute name="NAME" x="-104.4575" y="-21.59" size="1.27" layer="21" ratio="10"/>
+</element>
+<element name="C17" library="rcl" library_urn="urn:adsk.eagle:library:334" package="E3,5-10" package3d_urn="urn:adsk.eagle:package:23351/1" value="1uF 63V" x="-99.06" y="-35.56" smashed="yes">
+<attribute name="NAME" x="-94.996" y="-32.131" size="1.27" layer="25" ratio="10"/>
+<attribute name="POPULARITY" value="5" x="-99.06" y="-35.56" size="1.778" layer="27" display="off"/>
+<attribute name="SPICEPREFIX" value="C" x="-99.06" y="-35.56" size="1.778" layer="27" display="off"/>
+<attribute name="VALUE" x="-102.362" y="-38.608" size="1.27" layer="27" ratio="10"/>
+</element>
 </elements>
 <signals>
@@
 <contactref element="D10" pad="A"/>
 <contactref element="C16" pad="-"/>
+<contactref element="Q1I1" pad="1"/>
+<contactref element="C17" pad="-"/>
+<wire x1="-96.52" y1="-8.89" x2="-97.282" y2="-35.56" width="0" layer="19" extent="1-1"/>
+<wire x1="-82.042" y1="6.35" x2="-96.52" y2="-8.89" width="0" layer="19" extent="1-1"/>
+<wire x1="-85.09" y1="19.05" x2="-82.042" y2="6.35" width="0" layer="19" extent="1-1"/>
+<wire x1="-69.85" y1="19.05" x2="-85.09" y2="19.05" width="0" layer="19" extent="1-1"/>
+<wire x1="-62.23" y1="19.05" x2="-69.85" y2="19.05" width="0" layer="19" extent="1-1"/>
+<wire x1="-62.23" y1="30.48" x2="-62.23" y2="19.05" width="0" layer="19" extent="1-1"/>
+<wire x1="-67.31" y1="30.48" x2="-62.23" y2="30.48" width="0" layer="19" extent="1-1"/>
+<wire x1="-47.752" y1="20.32" x2="-62.23" y2="19.05" width="0" layer="19" extent="1-1"/>
+<wire x1="-33.782" y1="20.32" x2="-47.752" y2="20.32" width="0" layer="19" extent="1-1"/>
+<wire x1="-19.812" y1="20.32" x2="-33.782" y2="20.32" width="0" layer="19" extent="1-1"/>
+<wire x1="-80.01" y1="39.37" x2="-67.31" y2="30.48" width="0" layer="19" extent="1-1"/>
+<wire x1="2.54" y1="31.75" x2="-19.812" y2="20.32" width="0" layer="19" extent="1-1"/>
+<wire x1="5.08" y1="35.56" x2="2.54" y2="31.75" width="0" layer="19" extent="1-1"/>
+<wire x1="15.24" y1="39.37" x2="5.08" y2="35.56" width="0" layer="19" extent="1-1"/>
+<wire x1="22.86" y1="39.37" x2="15.24" y2="39.37" width="0" layer="19" extent="1-1"/>
+<wire x1="22.86" y1="31.75" x2="22.86" y2="39.37" width="0" layer="19" extent="1-1"/>
+<wire x1="22.86" y1="29.21" x2="22.86" y2="31.75" width="0" layer="19" extent="1-1"/>
+<wire x1="15.24" y1="31.75" x2="15.24" y2="39.37" width="0" layer="19" extent="1-1"/>
+<wire x1="31.75" y1="36.83" x2="22.86" y2="39.37" width="0" layer="19" extent="1-1"/>
+<wire x1="43.18" y1="36.83" x2="31.75" y2="36.83" width="0" layer="19" extent="1-1"/>
+<wire x1="50.8" y1="40.64" x2="43.18" y2="36.83" width="0" layer="19" extent="1-1"/>
+<wire x1="35.56" y1="58.42" x2="31.75" y2="36.83" width="0" layer="19" extent="1-1"/>
 <wire x1="27.94" y1="62.23" x2="35.56" y2="58.42" width="0" layer="19" extent="1-1"/>
 <wire x1="11.43" y1="64.77" x2="27.94" y2="62.23" width="0" layer="19" extent="1-1"/>
-<wire x1="31.75" y1="36.83" x2="35.56" y2="58.42" width="0" layer="19" extent="1-1"/>
-<wire x1="22.86" y1="39.37" x2="31.75" y2="36.83" width="0" layer="19" extent="1-1"/>
-<wire x1="22.86" y1="31.75" x2="22.86" y2="39.37" width="0" layer="19" extent="1-1"/>
-<wire x1="22.86" y1="29.21" x2="22.86" y2="31.75" width="0" layer="19" extent="1-1"/>
-<wire x1="15.24" y1="39.37" x2="22.86" y2="39.37" width="0" layer="19" extent="1-1"/>
-<wire x1="15.24" y1="31.75" x2="22.86" y2="31.75" width="0" layer="19" extent="1-1"/>
-<wire x1="5.08" y1="35.56" x2="15.24" y2="39.37" width="0" layer="19" extent="1-1"/>
-<wire x1="2.54" y1="31.75" x2="5.08" y2="35.56" width="0" layer="19" extent="1-1"/>
-<wire x1="43.18" y1="36.83" x2="31.75" y2="36.83" width="0" layer="19" extent="1-1"/>
-<wire x1="50.8" y1="40.64" x2="43.18" y2="36.83" width="0" layer="19" extent="1-1"/>
 <wire x1="-13.97" y1="46.99" x2="5.08" y2="35.56" width="0" layer="19" extent="1-1"/>
 <wire x1="-22.86" y1="46.99" x2="-13.97" y2="46.99" width="0" layer="19" extent="1-1"/>
@@
 <wire x1="-74.93" y1="71.12" x2="-52.07" y2="76.2" width="0" layer="19" extent="1-1"/>
 <wire x1="-87.63" y1="76.2" x2="-74.93" y2="71.12" width="0" layer="19" extent="1-1"/>
-<wire x1="-19.812" y1="20.32" x2="2.54" y2="31.75" width="0" layer="19" extent="1-1"/>
-<wire x1="-33.782" y1="20.32" x2="-19.812" y2="20.32" width="0" layer="19" extent="1-1"/>
-<wire x1="-47.752" y1="20.32" x2="-33.782" y2="20.32" width="0" layer="19" extent="1-1"/>
-<wire x1="-62.23" y1="19.05" x2="-47.752" y2="20.32" width="0" layer="19" extent="1-1"/>
-<wire x1="-69.85" y1="19.05" x2="-62.23" y2="19.05" width="0" layer="19" extent="1-1"/>
-<wire x1="-62.23" y1="30.48" x2="-62.23" y2="19.05" width="0" layer="19" extent="1-1"/>
-<wire x1="-67.31" y1="30.48" x2="-62.23" y2="30.48" width="0" layer="19" extent="1-1"/>
-<wire x1="-85.09" y1="19.05" x2="-69.85" y2="19.05" width="0" layer="19" extent="1-1"/>
-<wire x1="-82.042" y1="6.35" x2="-85.09" y2="19.05" width="0" layer="19" extent="1-1"/>
-<wire x1="-80.01" y1="39.37" x2="-67.31" y2="30.48" width="0" layer="19" extent="1-1"/>
 </signal>
 <signal name="N$2">
@@
 <wire x1="-37.338" y1="20.32" x2="-24.13" y2="60.96" width="0" layer="19" extent="1-1"/>
 </signal>
+<signal name="N$29">
+<contactref element="Q6" pad="S"/>
+<contactref element="R36" pad="1"/>
+<contactref element="R37" pad="1"/>
+<wire x1="-96.52" y1="-22.86" x2="-96.52" y2="-27.94" width="0" layer="19" extent="1-1"/>
+<wire x1="-80.01" y1="-2.54" x2="-96.52" y2="-22.86" width="0" layer="19" extent="1-1"/>
+</signal>
+<signal name="N$30">
+<contactref element="Q6" pad="G"/>
+<contactref element="R34" pad="2"/>
+<contactref element="R36" pad="2"/>
+<wire x1="-77.47" y1="-12.7" x2="-86.36" y2="-22.86" width="0" layer="19" extent="1-1"/>
+<wire x1="-85.09" y1="-2.54" x2="-77.47" y2="-12.7" width="0" layer="19" extent="1-1"/>
+</signal>
+<signal name="N$31">
+<contactref element="R34" pad="1"/>
+<contactref element="Q1I1" pad="3"/>
+<wire x1="-91.44" y1="-8.89" x2="-87.63" y2="-12.7" width="0" layer="19" extent="1-1"/>
+</signal>
+<signal name="N$32">
+<contactref element="Q6" pad="D"/>
+<contactref element="R35" pad="2"/>
+<wire x1="-82.55" y1="-2.54" x2="-86.36" y2="-17.78" width="0" layer="19" extent="1-1"/>
+</signal>
+<signal name="N$33">
+<contactref element="Q1I1" pad="2"/>
+<contactref element="R35" pad="1"/>
+<contactref element="SW1" pad="P$1"/>
+<contactref element="C17" pad="+"/>
+<wire x1="-101.6" y1="-25.4" x2="-100.838" y2="-35.56" width="0" layer="19" extent="1-1"/>
+<wire x1="-96.52" y1="-17.78" x2="-101.6" y2="-25.4" width="0" layer="19" extent="1-1"/>
+<wire x1="-93.98" y1="-8.89" x2="-96.52" y2="-17.78" width="0" layer="19" extent="1-1"/>
+</signal>
+<signal name="N$34">
+<contactref element="R37" pad="2"/>
+<contactref element="SW1" pad="P$2"/>
+<wire x1="-86.36" y1="-27.94" x2="-104.1" y2="-25.4" width="0" layer="19" extent="1-1"/>
+</signal>
 </signals>
