File: hardware/original design/tl494-orig.brd (EAGLE design)
At the start: 100 x 80 mm, 79 parts, among them IC1 TL494CN, J1 CON_HEADER_1X02-PTH, K2 24V, Q1 2N5551, Q1I 8050, Q1I1 2N3904, Q2 8550, Q2I 8050, Q3 8050, Q4 2SK4145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

Commit message: partial board placement and started fix on latch swith problem
Parts:
- removed J1: CON_HEADER_1X02-PTH, dp_devices.v6:M1X2
- removed K2: 24V, relay:G5LE
- removed OK1: PC817, optocoupler:DIL04
- removed T1: PAD_TERMINAL-1.02MM_ROUND, dp_devices.v6:CON_PAD_ROUND_1.02MM
- removed T3: PAD_TERMINAL-1.02MM_SQUARE, dp_devices.v6:CON_PAD_SQUARE_1.02MM
- added D6: ?, diode:DO35-10
- added K1: 24V, relay:G2R
- added Q5: 2SK4145, dp_devices.v6:TO-220V
- added R23, R24: 20K, rcl:0207/10
- added SW1: SW_MEMBRANE, dp_devices.v6:SW_MEMBRANE
- C10, C11: device rcl:E7,5-18 -> rcl:E3,5-10
- C12: device rcl:E5-13 -> rcl:E3,5-10
- C17: device rcl:E2-5 -> rcl:E3,5-10
- D3: value FCH30A06 -> (none)
- Q6: value IRF9540 -> IRF9530
- R20: value 1K -> 330R 1W
- R22: value 1K -> 2K
- moved C17 196.3 mm to (-99.1, -35.6), turned to 0 degrees
- moved R35 179.1 mm to (-91.4, -17.8), turned to 0 degrees
- moved Q1I1 167.8 mm to (-94.0, -8.89)
- moved Q6 162.6 mm to (-82.5, 0.00), turned to 0 degrees
- moved R34 158.2 mm to (-82.5, -12.7)
- moved R22 146.8 mm to (-82.5, 76.2)
- moved R20 141.6 mm to (-57.1, 76.2)
- moved R37 140.1 mm to (-91.4, -27.9)
- moved R36 139.5 mm to (-91.4, -22.9)
- moved D7 15.3 mm to (70.5, 4.70)
- moved R26 13.3 mm to (85.2, 5.46)
- moved C12 12.0 mm to (77.5, 59.7)
- moved D3 12.0 mm to (49.5, 54.6)
- moved R25 12.0 mm to (96.5, 54.6)
- moved L1 12.0 mm to (59.7, 63.5)
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Connections:
- removed net N$35: OK1.1, R22.1
- new net ACC: R24.2
- new net N$29: Q6.S, R36.1, R37.1
- new net VOUT_YELLOW: Q5.3, R22.2
- net +V: now also K1.P; no longer K2.P
- net GND: now also D6.A, R20.2, R22.1, R23.1; no longer OK1.2, T3.P
- net N$20: now also D6.C, Q5.1, R23.2, R24.1; no longer Q1I1.2, R20.1
- net N$23: now also K1.1; no longer K2.1
- net N$24: now also K1.2; no longer K2.2
- net N$32: no longer R26.2
- net N$33: now also Q1I1.2, SW1.P$1; no longer J1.1, R20.2, R22.2
- net N$34: now also SW1.P$2; no longer J1.2
- net VIN: now also K1.S, R26.2; no longer K2.S, Q6.S, R36.1, R37.1, T1.P
- net VOUT: now also Q5.2, R20.1
